File: pcb/tagconnect6p-2-jlink-interface/tagconnect6p-2-jlink-interface.kicad_sch (KiCad schematic)
At the start: 2 parts, among them J1 Conn_ARM_JTAG_SWD_20, J2 Conn_02x03_Counter_Clockwise

Commit message: Generate manuf files - ERROR in PCBA
Parts:
- J2: LCSC C11214 -> C11214
Changed lines of the file:
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@@
 			)
 		)
-		(property "LCSC" "C11214 "
+		(property "LCSC" "C11214"
 			(at 208.28 104.14 0)
 			(hide yes)
